File: CX_buttonlight.kicad_pcb (KiCad board)
At the start: 2 copper layers, 17 x 5.5 mm, 10 parts, among them U1 LM317L_SOT-89

Commit message: updated design (tweaks + specs), sent to JLCPCB
Parts:
- D4: value D -> BAS4002ARPPE6327HTSA1; footprint Diode_SMD:D_0603_1608Metric_Pad1.05x0.95mm_HandSolder -> EC-parts:BAS4002ARPPE6327HTSA1
- moved Ground1 16.0 mm to (100.7, 60.7)
- moved Supply1 16.0 mm to (100.7, 64.8)
- moved D4 10.6 mm to (103.2, 62.8), turned to 180 degrees
Connections:
- C1 pad 1: Net-(D4-K) -> Net-(D4-+)
- D4 pad 1: Net-(D4-K) -> GND
- Ground1 pad 1: GND -> Net-(D4-~_2)
- U1 pad 3: Net-(D4-K) -> Net-(D4-+)
Routing:
- net Net-(D4-+): track 0.00 -> 13.0 mm, vias 0 -> 1
- net Net-(D4-K): track 10.5 -> 0.00 mm, vias 1 -> 0
- net Net-(D4-~_2): track 0.00 -> 2.39 mm
- net Net-(U1-ADJ): track 10.7 -> 8.45 mm, vias 2 -> 0
- net Net-(D1-A): track 18.5 -> 16.8 mm
- net GND: track 21.9 -> 21.0 mm
- net Net-(D4-~_1): track 1.62 -> 2.37 mm
- added copper zone on B.Cu, net GND
- added copper zone on F.Cu, net Net-(D1-A)
- removed copper zone on B.Cu, net (none)

Commit message: Tweaks og tekster
Routing:
- net GND: track 21.0 -> 21.1 mm, vias 1 -> 2
Other:
- board text added: "PowerStation 2025 v1.2"
- board text removed: "PowerStation 2025 v1.1"
Changed lines of the file:
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@@
 		)
 		(fp_text user "${REFERENCE}"
-			(at 0.5 -6.9 270)
+			(at 0.5 -6.9 -90)
 			(layer "B.Fab")
 			(hide yes)
@@
 		)
 	)
-	(gr_text "PowerStation\n2025 v1.1"
+	(gr_text "PowerStation\n2025 v1.2"
 		(at 109.8 64.2 0)
 		(layer "B.SilkS")
@@
 	)
 	(segment
+		(start 103.85 65.1)
+		(end 104.05 65.1)
+		(width 0.2)
+		(layer "F.Cu")
+		(net 3)
+	)
+	(segment
+		(start 103.85 65.1)
+		(end 103.9 65.15)
+		(width 0.4)
+		(layer "F.Cu")
+		(net 3)
+	)
+	(segment
 		(start 112.25 65.15)
 		(end 112.3 65.2)
@@
 	)
 	(segment
+		(start 103.85 65.1)
+		(end 103.8 65.15)
+		(width 0.4)
+		(layer "F.Cu")
+		(net 3)
+	)
+	(segment
 		(start 116 63.775)
 		(end 116 64)
@@
 	(segment
 		(start 104.05 65.1)
-		(end 103.95 65.2)
-		(width 0.4)
+		(end 104.15 65.2)
+		(width 0.2)
 		(layer "F.Cu")
 		(net 3)
@@
 	)
 	(segment
-		(start 101.6 65.2)
-		(end 101 64.6)
-		(width 0.4)
-		(layer "F.Cu")
-		(net 3)
-	)
-	(segment
 		(start 108.5 65.1)
 		(end 108.6 65.2)
@@
 	)
 	(segment
+		(start 103.9 65.15)
+		(end 108.55 65.15)
+		(width 0.4)
+		(layer "F.Cu")
+		(net 3)
+	)
+	(segment
 		(start 114 65)
 		(end 114 63.7875)
@@
 	)
 	(segment
-		(start 104.15 65.2)
-		(end 104.05 65.1)
-		(width 0.2)
-		(layer "F.Cu")
-		(net 3)
-	)
-	(segment
-		(start 108.55 65.15)
-		(end 104.1 65.15)
-		(width 0.4)
-		(layer "F.Cu")
-		(net 3)
-	)
-	(segment
-		(start 104.1 65.15)
-		(end 104.05 65.1)
+		(start 101.55 65.15)
+		(end 101 64.6)
 		(width 0.4)
 		(layer "F.Cu")
@@
 	)
 	(segment
+		(start 103.8 65.15)
+		(end 101.55 65.15)
+		(width 0.4)
+		(layer "F.Cu")
+		(net 3)
+	)
+	(segment
 		(start 101 64.6)
 		(end 101 63.75)
@@
 		(net 3)
 	)
-	(segment
-		(start 103.95 65.2)
-		(end 101.6 65.2)
-		(width 0.4)
-		(layer "F.Cu")
-		(net 3)
-	)
 	(via
-		(at 104.05 65.1)
+		(at 112.25 65.15)
 		(size 0.6)
 		(drill 0.3)
+		(layers "F.Cu" "B.Cu")
+		(net 3)
+	)
+	(via
+		(at 103.85 65.1)
+		(size 0.6)
+		(drill 0.3)
