File: CX_buttonlight.kicad_sch (KiCad schematic)
At the start: 10 parts, among them U1 LM317L_SOT-89

Commit message: v1.1 - med beskyttelsesdiode
Parts:
- renumbered Ground to Ground1, Supply to Supply1
Changed lines of the file:
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@@
 		(on_board yes)
 		(dnp no)
-		(property "Reference" "Supply"
+		(property "Reference" "Supply1"
 			(at 73.152 59.69 90)
 			(effects
@@
 			(project ""
 				(path "/a6c7f972-13d1-471d-8078-ec61320b86a9"
-					(reference "Supply")
+					(reference "Supply1")
 					(unit 1)
 				)
@@
 		(on_board yes)
 		(dnp no)
-		(property "Reference" "Ground"
+		(property "Reference" "Ground1"
 			(at 80.01 66.04 90)
 			(effects
@@
 			(project "CX_buttonlight"
 				(path "/a6c7f972-13d1-471d-8078-ec61320b86a9"
-					(reference "Ground")
-					(unit 1)
-				)
+					(reference "Ground1")
+					(unit 1)
+				)

Commit message: updated design (tweaks + specs), sent to JLCPCB
Parts:
- removed D4: D, Diode_SMD:D_0603_1608Metric_Pad1.05x0.95mm_HandSolder, symbol Device:D
- added D4: BAS4002ARPPE6327HTSA1, BAS4002ARPPE6327HTSA1, symbol SamacSys_Parts:BAS4002ARPPE6327HTSA1
Connections:
- net GND: now also D4.1 (-); no longer Ground1.1
- net at Supply1.1: now also D4.3 (~_2)
- net at C1.1, U1.3 (VI): now also D4.4 (+)
- new net: D4.2 (~_1), Ground1.1
Other:
- moved on the sheet: C1, D1, D2, D3, R1, R2, U1

Commit message: Tweaks og tekster
Parts:
- R2: value 220R -> 560R
Other:
- note added: "Fejltilslutnings sikring"
- note added: "Lysgivere"
- note added: "R2 values: 560R - E12 conservative choice with minimal heat dissipation 576R - E96 more heat, a bit more light 590R - E96 even more heat, go no higher."
- note added: "Spændingsregulering"
- company: (none) -> PowerStation
- title: (none) -> CX vippeknap-lys
- moved on the sheet: C1, D1, D2, D3, D4, R1, R2, U1
